File: pure_kicad/charger.kicad_sch (KiCad schematic)
At the start: 96 parts, among them J1 XT30M, J2 XT30F, Q1 Q_NMOS_DGS, Q2 Q_NMOS_DGS, Q3 Q_NMOS_DGS, Q4 Q_NMOS_DGS, U1 BQ25756ERRVR

Commit message: Switch to single xt30 and JST B7B for pack, and add thermistor headers
Connections:
- net Earth: now also J1.1 (Pin_1), J2.1 (Pin_1); no longer J1.2 (Pin_2), J2.2 (Pin_2)
- net VAC: now also J1.2 (Pin_2); no longer J1.1 (Pin_1)
- net VCC: now also J2.2 (Pin_2); no longer J2.1 (Pin_1)
Changed lines of the file:
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@@
 	(symbol
 		(lib_id "Connector:Conn_01x02_Pin")
-		(at 36.83 33.02 0)
+		(at 36.83 35.56 0)
+		(mirror x)
 		(unit 1)
 		(exclude_from_sim no)
@@
 		(on_board yes)
 		(dnp no)
-		(fields_autoplaced yes)
 		(property "Reference" "J1"
-			(at 37.465 27.94 0)
+			(at 37.465 40.64 0)
 			(effects
 				(font
@@
 		)
 		(property "Value" "XT30M"
-			(at 37.465 30.48 0)
+			(at 37.465 38.1 0)
 			(effects
 				(font
@@
 		)
 		(property "Footprint" "cyberec:AMASS_XT30U-M_1x02_P5.0mm_Vertical"
-			(at 36.83 33.02 0)
+			(at 36.83 35.56 0)
 			(effects
 				(font
@@
 		)
 		(property "Datasheet" "~"
-			(at 36.83 33.02 0)
+			(at 36.83 35.56 0)
 			(effects
 				(font
@@
 		)
 		(property "Description" "Generic connector, single row, 01x02, script generated"
-			(at 36.83 33.02 0)
+			(at 36.83 35.56 0)
 			(effects
 				(font
@@
 	(symbol
 		(lib_id "Connector:Conn_01x02_Pin")
-		(at 43.18 165.1 0)
+		(at 43.18 167.64 0)
+		(mirror x)
 		(unit 1)
 		(exclude_from_sim no)
@@
 		(on_board yes)
 		(dnp no)
-		(fields_autoplaced yes)
 		(property "Reference" "J2"
-			(at 43.815 160.02 0)
+			(at 43.815 172.72 0)
 			(effects
 				(font
@@
 		)
 		(property "Value" "XT30F"
-			(at 43.815 162.56 0)
+			(at 43.815 170.18 0)
 			(effects
 				(font
@@
 		)
 		(property "Footprint" "cyberec:AMASS_XT30U-F_1x02_P5.0mm_Vertical"
-			(at 43.18 165.1 0)
+			(at 43.18 167.64 0)
 			(effects
 				(font
@@
 		)
 		(property "Datasheet" "~"
-			(at 43.18 165.1 0)
+			(at 43.18 167.64 0)
 			(effects
 				(font
@@
 		)
 		(property "Description" "Generic connector, single row, 01x02, script generated"
-			(at 43.18 165.1 0)
+			(at 43.18 167.64 0)
 			(effects
 				(font
